File: PCB/pcb_aime/pcb_aime.kicad_pcb (KiCad board)
At the start: 2 copper layers, 17 parts, among them J1 Pin ESP, J2 Pin Capteur, J4 Pin LoRa, U1 LTC1050ACN8_PBF

Commit message: Ajout du nodered qui affiche sur le dashboard un chart des valeurs de gaz, la dernière valeur connus et une notification en cas de dépassement d'une valeur limite
Other:
- board outline added: 53.1 x 58 mm
- board text added: "Louis Rousset Alix Chagot Clément Marce"
Changed lines of the file:
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@@
 		(tags "capacitor")
 		(property "Reference" "C5"
-			(at 2.75 0 360)
+			(at 2.75 0 0)
 			(layer "F.SilkS")
 			(effects
@@
 		(tags "resistor")
 		(property "Reference" "R2"
-			(at -3 0 360)
+			(at -3 0 0)
 			(layer "F.SilkS")
 			(effects
@@
 		)
 		(property "Value" "100k"
-			(at 0 1.65 360)
+			(at 0 1.65 0)
 			(layer "F.Fab")
 			(hide yes)
@@
 		(tags "resistor")
 		(property "Reference" "R1"
-			(at -3 0 360)
+			(at -3 0 0)
 			(layer "F.SilkS")
 			(effects
@@
 		)
 		(property "Value" "1k"
-			(at 0 1.65 360)
+			(at 0 1.65 0)
 			(layer "F.Fab")
 			(hide yes)
@@
 		(tags "capacitor")
 		(property "Reference" "C2"
-			(at 2.75 0 360)
+			(at 2.75 0 0)
 			(layer "F.SilkS")
 			(effects
@@
 		(tags "capacitor")
 		(property "Reference" "C1"
-			(at 2.75 0 360)
+			(at 2.75 0 0)
 			(layer "F.SilkS")
 			(effects
@@
 		(tags "capacitor")
 		(property "Reference" "C3"
-			(at 2.75 0 360)
+			(at 2.75 0 0)
 			(layer "F.SilkS")
 			(effects
@@
 		(tags "resistor")
 		(property "Reference" "R3"
-			(at -3 0 360)
+			(at -3 0 0)
 			(layer "F.SilkS")
 			(effects
@@
 		)
 		(property "Value" "10k"
-			(at 0 1.65 360)
+			(at 0 1.65 0)
 			(layer "F.Fab")
 			(hide yes)
@@
 		)
 		(fp_text user "${REFERENCE}"
-			(at 0 5.08 360)
+			(at 0 5.08 0)
 			(layer "F.Fab")
 			(effects
@@
 		(tags "resistor")
 		(property "Reference" "R4"
-			(at -3 0 360)
+			(at -3 0 0)
 			(layer "F.SilkS")
 			(effects
@@
 		)
 		(property "Value" "100k"
-			(at 0 1.65 360)
+			(at 0 1.65 0)
 			(layer "F.Fab")
 			(hide yes)
@@
 		(tags "resistor")
 		(property "Reference" "R6"
-			(at -3 0 360)
+			(at -3 0 0)
 			(layer "F.SilkS")
 			(effects
@@
 		)
 		(property "Value" "1k"
-			(at 0 1.65 360)
+			(at 0 1.65 0)
 			(layer "F.Fab")
 			(hide yes)
@@
 		)
 	)
+	(gr_rect
+		(start 50.5 40.2)
+		(end 103.603867 98.203867)
+		(stroke
+			(width 0.05)
+			(type default)
+		)
+		(fill none)
+		(layer "Edge.Cuts")
+	)
+	(gr_text "Louis Rousset\nAlix Chagot\nClément Marce"
+		(at 94.2 44.9 0)
+		(layer "F.Cu")
+		(effects
+			(font
+				(size 0.7 0.7)
+				(thickness 0.175)
+				(bold yes)
+			)
+			(justify left bottom)
+		)
+	)
